Commit message: feat: Archivos .xacro
Co-authored-by: Copilot <copilot@github.com>

File: robx7_description/urdf/joystick.urdf (robot description, URDF)
Before this commit: robot robx7, 3 links, 2 joints
Joints:
- joint base_first_joint: axis 0 1 0 -> 0 0 1; origin xyz=0.0 0.0 0.1 rpy=0.0 0.0 0.0 -> xyz=0.0 0.0 0.1 rpy=-1.5708 -1.5708 0.0
- joint first_second_joint: origin xyz=0.0 0.0 0.3 rpy=0.0 0.0 0.0 -> xyz=0.3 0.0 0.0 rpy=1.5708 0.0 1.5708
