Commit message: fix: Añadido el gripper correctamente
Co-authored-by: Copilot <copilot@github.com>

File: robx7_description/urdf/robx7.urdf.xacro (robot description, xacro)
@@ -3,4 +3,4 @@
     <xacro:include filename="common_properties.xacro"/>
     <xacro:include filename="robx7_arm.xacro"/>
-    <!-- <xacro:include filename="robx7_gripper.xacro"/> -->
+    <xacro:include filename="robx7_gripper.xacro"/>
 </robot>

File: robx7_description/urdf/robx7_gripper.xacro (robot description, xacro)
@@ -1,10 +1,10 @@
 <?xml version="1.0"?>
 <robot xmlns:xacro="http://www.ros.org/wiki/xacro">
-    <xacro:property name="gripper_base_length" value="0.1"/>
-    <xacro:property name="gripper_base_width" value="0.05"/>
-    <xacro:property name="gripper_base_height" value="0.02"/>
-    <xacro:property name="gripper_finger_length" value="0.05"/>
-    <xacro:property name="gripper_finger_width" value="0.02"/>
-    <xacro:property name="gripper_finger_height" value="0.02"/>
+    <xacro:property name="gripper_base_length" value="0.05"/>
+    <xacro:property name="gripper_base_width" value="0.2"/>
+    <xacro:property name="gripper_base_height" value="0.1"/>
+    <xacro:property name="gripper_finger_length" value="0.15"/>
+    <xacro:property name="gripper_finger_width" value="0.08"/>
+    <xacro:property name="gripper_finger_height" value="0.03"/>
     <link name="gripper_base">
         <visual>
@@ -37,19 +37,20 @@
         <parent link="third_link"/>
         <child link="gripper_base"/>
-        <origin xyz="${third_link_length/2} 0 0" rpy="0.0 0.0 0.0"/>
+        <origin xyz="${third_link_length} 0 0" rpy="${PI/2} 0.0 0.0"/>
     </joint>
-    <!-- <joint name="gripper_base_finger_left" type="prismatic">
+    <joint name="gripper_base_finger_left" type="prismatic">
         <parent link="gripper_base"/>
         <child link="gripper_finger_left"/>
-        <origin xyz="${gripper_base_length/2} ${gripper_base_width/2} 0" rpy="0.0 0.0 0.0"/>
+        <origin xyz="${gripper_base_length/2} ${gripper_base_width/2-gripper_finger_height/2} 0" rpy="${PI/2} 0.0 0.0"/>
         <axis xyz="0 0 1"/>
-        <limit lower="0.0" upper="${gripper_base_length/2}" effort="1" velocity="1"/>
+        <limit lower="0.0" upper="${gripper_base_width/2-gripper_finger_height}" effort="${effort}" velocity="${velocity}"/>
     </joint>
     <joint name="gripper_base_finger_right" type="prismatic">
         <parent link="gripper_base"/>
         <child link="gripper_finger_right"/>
-        <origin xyz="${gripper_base_length/2} $-{gripper_base_width/2} 0" rpy="0.0 0.0 0.0"/>
+        <origin xyz="${gripper_base_length/2} -${gripper_base_width/2-gripper_finger_height/2} 0" rpy="-${PI/2} 0.0 0.0"/>
         <axis xyz="0 0 1"/>
-        <limit lower="0" upper="-${gripper_base_length/2}" effort="1" velocity="1"/>
-    </joint> -->
+        <limit lower="0.0" upper="${gripper_base_width/2-gripper_finger_height}" effort="${effort}" velocity="${velocity}"/>
+        <mimic joint="gripper_base_finger_left" multiplier="1.0" offset="0.0"/>
+    </joint>
 </robot>
