Commit message: feat: Visualizacion del robot en Rviz
Co-authored-by: Copilot <copilot@github.com>

File: robx7_description/urdf/robx7_gripper.xacro (robot description, xacro)
@@ -49,8 +49,8 @@
         <parent link="gripper_base"/>
         <child link="gripper_finger_right"/>
-        <origin xyz="${gripper_base_length/2} -${gripper_base_width/2-gripper_finger_height/2} 0" rpy="-${PI/2} 0.0 0.0"/>
+        <origin xyz="${gripper_base_length/2} -${gripper_base_width/2-gripper_finger_height/2} 0" rpy="${PI/2} 0.0 0.0"/>
         <axis xyz="0 0 1"/>
         <limit lower="0.0" upper="${gripper_base_width/2-gripper_finger_height}" effort="${effort}" velocity="${velocity}"/>
-        <mimic joint="gripper_base_finger_left" multiplier="1.0" offset="0.0"/>
+        <mimic joint="gripper_base_finger_left" multiplier="-1.0" offset="0.0"/>
     </joint>
 </robot>
