Commit message: feat: Add launch file and update dependencies for robot simulation
Co-authored-by: Copilot <copilot@github.com>

File: robx7_description/urdf/common_properties.xacro (robot description, xacro)
@@ -10,3 +10,33 @@
         <color rgba="0.5 0.5 0.5 1"/>
     </material>
+        <xacro:macro name="box_inertia" params="m x y z">
+        <inertal>
+            <mass value="${m}"/>
+            <origin xyz="0.0 0.0 ${z/2}" rpy="0.0 0.0 0.0"/>
+            <inertia
+                ixx = "${m/12)*(z*z + y*y)}" ixy = "0" ixz = "0"
+                iyy = "${m/12)*(x*x + z*z)}" iyz = "0"
+                izz = "${m/12)*(x*x + y*y)}"/>
+        </inertal>
+    </xacro:macro>
+    <xacro:macro name="cylinder_inertia" params="m r l">
+        <inertal>
+            <mass value="${m}"/>
+            <origin xyz="0.0 0.0 ${l/2}" rpy="0.0 0.0 0.0"/>
+            <inertia
+                ixx = "${m/12)*(3*r*r + l*l)}" ixy = "0" ixz = "0"
+                iyy = "${m/12)*(3*r*r + l*l)}" iyz = "0"
+                izz = "${m/2)*(r*r)}"/>
+        </inertal>
+    </xacro:macro>
+    <xacro:macro name="sphere_inertia" params="m r">
+        <inertal>
+            <mass value="${m}"/>
+            <origin xyz="0.0 0.0 ${r}" rpy="0.0 0.0 0.0"/>
+            <inertia
+                ixx = "${(2/5)*m*r*r}" ixy = "0" ixz = "0"
+                iyy = "${(2/5)*m*r*r}" iyz = "0"
+                izz = "${(2/5)*m*r*r}"/>
+        </inertal>
+    </xacro:macro>
 </robot>

File: robx7_description/urdf/robx7_arm.xacro (robot description, xacro)
@@ -6,8 +6,11 @@
     <xacro:property name="firts_link_length" value="0.1"/>
     <xacro:property name="firts_link_radius" value="0.05"/>
+    <xacro:property name="first_link_mass" value="1.0"/>
     <xacro:property name="second_link_length" value="0.4"/>
     <xacro:property name="second_link_radius" value="0.05"/>
+    <xacro:property name="second_link_mass" value="1.0"/>
     <xacro:property name="third_link_length" value="0.3"/>
     <xacro:property name="third_link_radius" value="0.05"/>
+    <xacro:property name="third_link_mass" value="1.0"/>
     <link name="base_link">
         <visual>
@@ -18,4 +21,11 @@
             <material name="gray"/>
         </visual>
+        <xacro:macro name="box_inertia" params="${base_link_mass} ${base_link_length} ${base_link_width} ${base_link_height}"/>
+        <collision>
+            <origin xyz="0.0 0.0 ${base_link_height/2}" rpy="0.0 0.0 0.0"/>
+            <geometry>
+                <box size="${base_link_length*0.8} ${base_link_width*0.8} ${base_link_height*0.8}"/>
+            </geometry>
+        </collision>
     </link>
      <link name="first_link">
@@ -27,4 +37,11 @@
             <material name="blue"/>
         </visual>
+        <xacro:macro name="cylinder_inertia" params="${first_link_mass} ${firts_link_radius} ${firts_link_length}"/>
+        <collision>
+            <origin xyz="0.0 0.0 ${firts_link_length/2}" rpy="0.0 0.0 0.0"/>
+            <geometry>
+                <cylinder radius="${firts_link_radius}" length="${firts_link_length}"/>
+            </geometry>
+        </collision>
     </link>
     <link name="second_link">
@@ -36,4 +53,11 @@
             <material name="gray"/>
         </visual>
+        <xacro:macro name="cylinder_inertia" params="${second_link_mass} ${second_link_radius} ${second_link_length}"/>
+        <collision>
+            <origin xyz="${second_link_length/2} 0.0 0.0" rpy="0.0 ${PI/2} 0.0"/>
+            <geometry>
+                <cylinder radius="${second_link_radius}" length="${second_link_length}"/>
+            </geometry>
+        </collision>
     </link>
     <link name="third_link">
@@ -45,4 +69,11 @@
             <material name="blue"/>
         </visual>
+        <xacro:macro name="cylinder_inertia" params="${third_link_mass} ${third_link_radius} ${third_link_length}"/>
+        <collision>
+            <origin xyz="${third_link_length/2} 0.0 0.0" rpy="0.0 ${PI/2} 0.0"/>
+            <geometry>
+                <cylinder radius="${third_link_radius}" length="${third_link_length}"/>
+            </geometry>
+        </collision>
     </link>
     <joint name="base_first_joint" type="revolute">

File: robx7_description/urdf/robx7_gripper.xacro (robot description, xacro)
@@ -4,7 +4,9 @@
     <xacro:property name="gripper_base_width" value="0.2"/>
     <xacro:property name="gripper_base_height" value="0.1"/>
+    <xacro:property name="gripper_base_mass" value="1.0"/>
     <xacro:property name="gripper_finger_length" value="0.15"/>
     <xacro:property name="gripper_finger_width" value="0.08"/>
     <xacro:property name="gripper_finger_height" value="0.03"/>
+    <xacro:property name="gripper_finger_mass" value="1.0"/>
     <link name="gripper_base">
         <visual>
@@ -15,4 +17,12 @@
             <material name="gray"/>
         </visual>
+        <xacro:macro name="box_inertia" params="${gripper_base_mass} ${gripper_base_length} ${gripper_base_width} ${gripper_base_height}"/>
+        <collision>
+            <origin xyz="0 0 0" rpy="0.0 0.0 0.0"/>
+            <geometry>
+                <box size="${gripper_base_length} ${gripper_base_width} ${gripper_base_height}"/>
+            </geometry>
+            <material name="gray"/>
+        </collision>
     </link>
     <link name="gripper_finger_left">
@@ -24,4 +34,11 @@
             <material name="blue"/>
         </visual>
+        <xacro:macro name="box_inertia" params="${gripper_finger_mass} ${gripper_finger_length} ${gripper_finger_width} ${gripper_finger_height}"/>
+        <collision>
+            <origin xyz="${gripper_finger_length/2} 0 0" rpy="0.0 0.0 0.0"/>
+            <geometry>
+                <box size="${gripper_finger_length} ${gripper_finger_width} ${gripper_finger_height}"/>
+            </geometry>
+        </collision>
     </link>
     <link name="gripper_finger_right">
@@ -33,4 +50,11 @@
             <material name="blue"/>
         </visual>
+        <xacro:macro name="box_inertia" params="${gripper_finger_mass} ${gripper_finger_length} ${gripper_finger_width} ${gripper_finger_height}"/>
+        <collision>
+            <origin xyz="${gripper_finger_length/2} 0 0" rpy="0.0 0.0 0.0"/>
+            <geometry>
+                <box size="${gripper_finger_length} ${gripper_finger_width} ${gripper_finger_height}"/>
+            </geometry>
+        </collision>
     </link>
     <joint name="third_link_gripper_base" type="fixed">
