Commit message: feat: Clase 26 octubre

File: robx7_description/urdf/common_properties.xacro (robot description, xacro)
@@ -10,33 +10,33 @@
         <color rgba="0.5 0.5 0.5 1"/>
     </material>
-        <xacro:macro name="box_inertia" params="m x y z">
-        <inertal>
+    <xacro:macro name="box_inertia" params="m x y z o_xyz o_rpy">
+        <inertial>
             <mass value="${m}"/>
-            <origin xyz="0.0 0.0 ${z/2}" rpy="0.0 0.0 0.0"/>
+            <origin xyz="${o_xyz}" rpy="${o_rpy}"/>
             <inertia
-                ixx = "${m/12)*(z*z + y*y)}" ixy = "0" ixz = "0"
-                iyy = "${m/12)*(x*x + z*z)}" iyz = "0"
-                izz = "${m/12)*(x*x + y*y)}"/>
-        </inertal>
+                ixx = "${(m/12)*(z*z + y*y)}" ixy = "0" ixz = "0"
+                iyy = "${(m/12)*(x*x + z*z)}" iyz = "0"
+                izz = "${(m/12)*(x*x + y*y)}"/>
+        </inertial>
     </xacro:macro>
-    <xacro:macro name="cylinder_inertia" params="m r l">
-        <inertal>
+    <xacro:macro name="cylinder_inertia" params="m r l o_xyz o_rpy">
+        <inertial>
             <mass value="${m}"/>
-            <origin xyz="0.0 0.0 ${l/2}" rpy="0.0 0.0 0.0"/>
+            <origin xyz="${o_xyz}" rpy="${o_rpy}"/>
             <inertia
-                ixx = "${m/12)*(3*r*r + l*l)}" ixy = "0" ixz = "0"
-                iyy = "${m/12)*(3*r*r + l*l)}" iyz = "0"
-                izz = "${m/2)*(r*r)}"/>
-        </inertal>
+                ixx = "${(m/12)*(3*r*r + l*l)}" ixy = "0" ixz = "0"
+                iyy = "${(m/12)*(3*r*r + l*l)}" iyz = "0"
+                izz = "${(m/2)*(r*r)}"/>
+        </inertial>
     </xacro:macro>
-    <xacro:macro name="sphere_inertia" params="m r">
-        <inertal>
+    <xacro:macro name="sphere_inertia" params="m r o_xyz">
+        <inertial>
             <mass value="${m}"/>
-            <origin xyz="0.0 0.0 ${r}" rpy="0.0 0.0 0.0"/>
+            <origin xyz="${o_xyz}" rpy="0.0 0.0 0.0"/>
             <inertia
                 ixx = "${(2/5)*m*r*r}" ixy = "0" ixz = "0"
                 iyy = "${(2/5)*m*r*r}" iyz = "0"
                 izz = "${(2/5)*m*r*r}"/>
-        </inertal>
+        </inertial>
     </xacro:macro>
 </robot>

File: robx7_description/urdf/robx7.urdf.xacro (robot description, xacro)
@@ -4,3 +4,4 @@
     <xacro:include filename="robx7_arm.xacro"/>
     <xacro:include filename="robx7_gripper.xacro"/>
+    <xacro:include filename="robx7_gazebo.xacro"/>
 </robot>

File: robx7_description/urdf/robx7_arm.xacro (robot description, xacro)
@@ -4,4 +4,5 @@
     <xacro:property name="base_link_width" value="0.3"/>
     <xacro:property name="base_link_height" value="0.1"/>
+    <xacro:property name="base_link_mass" value="0.1"/>
     <xacro:property name="firts_link_length" value="0.1"/>
     <xacro:property name="firts_link_radius" value="0.05"/>
@@ -10,7 +11,10 @@
     <xacro:property name="second_link_radius" value="0.05"/>
     <xacro:property name="second_link_mass" value="1.0"/>
+    <xacro:property name="second_link_rpy" value="0.0 ${PI/2} 0.0"/>
     <xacro:property name="third_link_length" value="0.3"/>
     <xacro:property name="third_link_radius" value="0.05"/>
     <xacro:property name="third_link_mass" value="1.0"/>
+    <xacro:property name="third_link_rpy" value="0.0 ${PI/2} 0.0"/>
+    <link name="world"/>
     <link name="base_link">
         <visual>
@@ -21,9 +25,9 @@
             <material name="gray"/>
         </visual>
-        <xacro:macro name="box_inertia" params="${base_link_mass} ${base_link_length} ${base_link_width} ${base_link_height}"/>
+        <xacro:box_inertia m="${base_link_mass}" x="${base_link_length}" y="${base_link_width}" z="${base_link_height}" o_xyz="0.0 0.0 ${base_link_height/2}" o_rpy="0.0 0.0 0.0"/>
         <collision>
             <origin xyz="0.0 0.0 ${base_link_height/2}" rpy="0.0 0.0 0.0"/>
             <geometry>
-                <box size="${base_link_length*0.8} ${base_link_width*0.8} ${base_link_height*0.8}"/>
+                <box size="${base_link_length} ${base_link_width} ${base_link_height}"/>
             </geometry>
         </collision>
@@ -37,5 +41,5 @@
             <material name="blue"/>
         </visual>
-        <xacro:macro name="cylinder_inertia" params="${first_link_mass} ${firts_link_radius} ${firts_link_length}"/>
+        <xacro:cylinder_inertia m="${first_link_mass}" r="${firts_link_radius}" l="${firts_link_length}" o_xyz="0.0 0.0 ${firts_link_length/2}" o_rpy="0.0 0.0 0.0"/>
         <collision>
             <origin xyz="0.0 0.0 ${firts_link_length/2}" rpy="0.0 0.0 0.0"/>
@@ -47,5 +51,5 @@
     <link name="second_link">
         <visual>
-            <origin xyz="${second_link_length/2} 0.0 0.0" rpy="0.0 ${PI/2} 0.0"/>
+            <origin xyz="${second_link_length/2} 0.0 0.0" rpy="${second_link_rpy}"/>
             <geometry>
                 <cylinder radius="${second_link_radius}" length="${second_link_length}"/>
@@ -53,7 +57,7 @@
             <material name="gray"/>
         </visual>
-        <xacro:macro name="cylinder_inertia" params="${second_link_mass} ${second_link_radius} ${second_link_length}"/>
+        <xacro:cylinder_inertia m="${second_link_mass}" r="${second_link_radius}" l="${second_link_length}" o_xyz="${second_link_length/2} 0.0 0.0" o_rpy="${second_link_rpy}"/>
         <collision>
-            <origin xyz="${second_link_length/2} 0.0 0.0" rpy="0.0 ${PI/2} 0.0"/>
+            <origin xyz="${second_link_length/2} 0.0 0.0" rpy="${second_link_rpy}"/>
             <geometry>
                 <cylinder radius="${second_link_radius}" length="${second_link_length}"/>
@@ -63,5 +67,5 @@
     <link name="third_link">
         <visual>
-            <origin xyz="${third_link_length/2} 0.0 0.0" rpy="0.0 ${PI/2} 0.0"/>
+            <origin xyz="${third_link_length/2} 0.0 0.0" rpy="${third_link_rpy}"/>
             <geometry>
                 <cylinder radius="${third_link_radius}" length="${third_link_length}"/>
@@ -69,7 +73,7 @@
             <material name="blue"/>
         </visual>
-        <xacro:macro name="cylinder_inertia" params="${third_link_mass} ${third_link_radius} ${third_link_length}"/>
+        <xacro:cylinder_inertia m="${third_link_mass}" r="${third_link_radius}" l="${third_link_length}" o_xyz="${third_link_length/2} 0.0 0.0" o_rpy="${third_link_rpy}"/>
         <collision>
-            <origin xyz="${third_link_length/2} 0.0 0.0" rpy="0.0 ${PI/2} 0.0"/>
+            <origin xyz="${third_link_length/2} 0.0 0.0" rpy="${third_link_rpy}"/>
             <geometry>
                 <cylinder radius="${third_link_radius}" length="${third_link_length}"/>
@@ -77,4 +81,9 @@
         </collision>
     </link>
+    <joint name="world_base_joint" type="fixed">
+        <parent link="world"/>
+        <child link="base_link"/>
+        <origin xyz="0.0 0.0 0.0" rpy="0.0 0.0 0.0"/>
+    </joint>
     <joint name="base_first_joint" type="revolute">
         <parent link="base_link"/>

File: robx7_description/urdf/robx7_gazebo.xacro (robot description, xacro)
@@ -1,3 +1,11 @@
-<gazebo reference="base_link">
-  <material>Gazebo/Blue</material>
-</gazebo>
+<?xml version="1.0"?>
+<robot xmlns:xacro="http://www.ros.org/wiki/xacro">
+  <gazebo>
+    <plugin filename="libgazebo_ros_joint_state_publisher.so" name="gazebo_ros_joint_state_publisher">
+      <ros>
+        <namespace>/</namespace>
+      </ros>
+      <publish_rate>50.0</publish_rate>
+    </plugin>
+  </gazebo>
+</robot>

File: robx7_description/urdf/robx7_gripper.xacro (robot description, xacro)
@@ -5,8 +5,10 @@
     <xacro:property name="gripper_base_height" value="0.1"/>
     <xacro:property name="gripper_base_mass" value="1.0"/>
+    <xacro:property name="gripper_base_rpy" value="0.0 0.0 0.0"/>
     <xacro:property name="gripper_finger_length" value="0.15"/>
     <xacro:property name="gripper_finger_width" value="0.08"/>
     <xacro:property name="gripper_finger_height" value="0.03"/>
     <xacro:property name="gripper_finger_mass" value="1.0"/>
+    <xacro:property name="gripper_finger_rpy" value="0.0 0.0 0.0"/>
     <link name="gripper_base">
         <visual>
@@ -17,5 +19,5 @@
             <material name="gray"/>
         </visual>
-        <xacro:macro name="box_inertia" params="${gripper_base_mass} ${gripper_base_length} ${gripper_base_width} ${gripper_base_height}"/>
+        <xacro:box_inertia m="${gripper_base_mass}" x="${gripper_base_length}" y="${gripper_base_width}" z="${gripper_base_height}" o_xyz="0.0 0.0 0.0" o_rpy="0.0 0.0 0.0"/>
         <collision>
             <origin xyz="0 0 0" rpy="0.0 0.0 0.0"/>
@@ -34,5 +36,5 @@
             <material name="blue"/>
         </visual>
-        <xacro:macro name="box_inertia" params="${gripper_finger_mass} ${gripper_finger_length} ${gripper_finger_width} ${gripper_finger_height}"/>
+        <xacro:box_inertia m="${gripper_finger_mass}" x="${gripper_finger_length}" y="${gripper_finger_width}" z="${gripper_finger_height}" o_xyz="${gripper_finger_length/2} 0 0" o_rpy="0.0 0.0 0.0"/>
         <collision>
             <origin xyz="${gripper_finger_length/2} 0 0" rpy="0.0 0.0 0.0"/>
@@ -50,5 +52,5 @@
             <material name="blue"/>
         </visual>
-        <xacro:macro name="box_inertia" params="${gripper_finger_mass} ${gripper_finger_length} ${gripper_finger_width} ${gripper_finger_height}"/>
+        <xacro:box_inertia m="${gripper_finger_mass}" x="${gripper_finger_length}" y="${gripper_finger_width}" z="${gripper_finger_height}" o_xyz="${gripper_finger_length/2} 0 0" o_rpy="0.0 0.0 0.0"/>
         <collision>
             <origin xyz="${gripper_finger_length/2} 0 0" rpy="0.0 0.0 0.0"/>
